File: Mjolnir-PCB/Mjolnir.brd (EAGLE design)
At the start: 53 x 17.8 mm, 14 parts, among them U1 ATTINY85-20PU, U2 L78M09ABDT-TR, X1 USB-A

Commit message: Replaced zener diodes to SOD-123 footprint
Parts:
- removed D1, D2: 3.6 Zener, microbuilder:SMADIODE
- added D4, D5: BZT52C3V9-7-F, BZT52C3V9-7-F:SOD3715X145N
Connections:
- net GND: now also D4.A, D5.A; no longer D1.A, D2.A
- net N$3: now also D5.C; no longer D1.C
- net N$5: now also D4.C; no longer D2.C
Routing:
- net N$3: track 25.6 -> 20.9 mm
- net N$5: track 19.4 -> 18.8 mm
Changed lines of the file:
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@@
 </element>
 <element name="ISP1" library="adafruit" library_urn="urn:adsk.eagle:library:420" package="AVRISP" package3d_urn="urn:adsk.eagle:package:6240744/1" value="AVRISP-6" x="48.26" y="8.89" smashed="yes"/>
-<element name="D1" library="microbuilder" package="SMADIODE" value="3.6 Zener" x="22.86" y="14.605" smashed="yes">
-<attribute name="VALUE" x="20.32" y="12.319" size="0.4064" layer="27" font="vector" ratio="10"/>
-</element>
-<element name="D2" library="microbuilder" package="SMADIODE" value="3.6 Zener" x="22.86" y="2.54" smashed="yes">
-<attribute name="VALUE" x="20.32" y="0.254" size="0.4064" layer="27" font="vector" ratio="10"/>
-</element>
 <element name="R1" library="adafruit" library_urn="urn:adsk.eagle:library:420" package="R0805" package3d_urn="urn:adsk.eagle:package:6240566/1" value="66.5" x="12.7" y="12.7" smashed="yes">
 <attribute name="VALUE" x="11.938" y="10.414" size="1.27" layer="27"/>
@@
 <attribute name="VALUE" x="20.86" y="4.255" size="1.27" layer="27" align="top-left"/>
 </element>
+<element name="D4" library="BZT52C3V9-7-F" package="SOD3715X145N" value="BZT52C3V9-7-F" x="21.59" y="2.54" smashed="yes">
+<attribute name="AVAILABILITY" value="In Stock" x="21.59" y="2.54" size="1.778" layer="27" display="off"/>
+<attribute name="DESCRIPTION" value=" Zener Diode 3.9V 500mW ±5% Surface Mount SOD-123 " x="21.59" y="2.54" size="1.778" layer="27" display="off"/>
+<attribute name="MF" value="Diodes Inc." x="21.59" y="2.54" size="1.778" layer="27" display="off"/>
+<attribute name="MP" value="BZT52C3V9-7-F" x="21.59" y="2.54" size="1.778" layer="27" display="off"/>
+<attribute name="NAME" x="19.39" y="3.84" size="0.8128" layer="25"/>
+<attribute name="PACKAGE" value="SOD-123 Fairchild Semiconductor" x="21.59" y="2.54" size="1.778" layer="27" display="off"/>
+<attribute name="PRICE" value="None" x="21.59" y="2.54" size="1.778" layer="27" display="off"/>
+<attribute name="VALUE" x="19.39" y="1.24" size="0.8128" layer="27" align="top-left"/>
+</element>
+<element name="D5" library="BZT52C3V9-7-F" package="SOD3715X145N" value="BZT52C3V9-7-F" x="17.145" y="15.24" smashed="yes">
+<attribute name="AVAILABILITY" value="In Stock" x="17.145" y="15.24" size="1.778" layer="27" display="off"/>
+<attribute name="DESCRIPTION" value=" Zener Diode 3.9V 500mW ±5% Surface Mount SOD-123 " x="17.145" y="15.24" size="1.778" layer="27" display="off"/>
+<attribute name="MF" value="Diodes Inc." x="17.145" y="15.24" size="1.778" layer="27" display="off"/>
+<attribute name="MP" value="BZT52C3V9-7-F" x="17.145" y="15.24" size="1.778" layer="27" display="off"/>
+<attribute name="NAME" x="14.945" y="16.54" size="0.8128" layer="25"/>
+<attribute name="PACKAGE" value="SOD-123 Fairchild Semiconductor" x="17.145" y="15.24" size="1.778" layer="27" display="off"/>
+<attribute name="PRICE" value="None" x="17.145" y="15.24" size="1.778" layer="27" display="off"/>
+<attribute name="VALUE" x="14.945" y="13.94" size="0.8128" layer="27" align="top-left"/>
+</element>
 </elements>
 <signals>
@@
 </polygon>
 <contactref element="X1" pad="4"/>
-<contactref element="D1" pad="A"/>
-<contactref element="D2" pad="A"/>
 <contactref element="ISP1" pad="6"/>
 <contactref element="U2" pad="2"/>
+<contactref element="D5" pad="A"/>
+<contactref element="D4" pad="A"/>
+<wire x1="23.27" y1="2.54" x2="18.825" y2="15.24" width="0" layer="19" extent="1-1"/>
+<wire x1="6.41" y1="12.39" x2="23.27" y2="2.54" width="0" layer="19" extent="1-1"/>
 </signal>
 <signal name="+5V">
@@
 <signal name="N$3">
 <contactref element="X1" pad="2"/>
-<contactref element="D1" pad="C"/>
 <contactref element="R1" pad="1"/>
 <contactref element="R3" pad="2"/>
@@
 <wire x1="8.89" y1="6.985" x2="7.315" y2="6.985" width="0.2032" layer="1"/>
 <wire x1="7.315" y1="6.985" x2="6.41" y2="7.89" width="0.2032" layer="1"/>
-<wire x1="20.5105" y1="14.605" x2="13.605" y2="14.605" width="0.2032" layer="1"/>
-<wire x1="13.605" y1="14.605" x2="11.7" y2="12.7" width="0.2032" layer="1"/>
+<contactref element="D5" pad="C"/>
+<wire x1="14.24" y1="15.24" x2="15.465" y2="15.24" width="0.2032" layer="1"/>
+<wire x1="11.7" y1="12.7" x2="14.24" y2="15.24" width="0.2032" layer="1"/>
 </signal>
 <signal name="N$5">
 <contactref element="X1" pad="3"/>
-<contactref element="D2" pad="C"/>
 <contactref element="R2" pad="1"/>
-<wire x1="20.5105" y1="2.54" x2="18.415" y2="2.54" width="0.2032" layer="1"/>
 <wire x1="18.415" y1="2.54" x2="16.51" y2="4.445" width="0.2032" layer="1"/>
 <wire x1="16.51" y1="7.62" x2="15.24" y2="8.89" width="0.2032" layer="1"/>
@@
 <wire x1="6.68" y1="10.16" x2="6.41" y2="9.89" width="0.2032" layer="1"/>
 <wire x1="11.7" y1="10.16" x2="6.68" y2="10.16" width="0.2032" layer="1"/>
+<contactref element="D4" pad="C"/>
+<wire x1="19.91" y1="2.54" x2="18.415" y2="2.54" width="0.2032" layer="1"/>
 </signal>
 <signal name="N$2">

Commit message: Updated PCB files
Routing:
- net +5V: track 75.8 -> 66.4 mm
- net N$3: track 20.9 -> 24.9 mm
- net N$5: track 18.8 -> 21.8 mm
Changed lines of the file:
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@@
 <drawing>
 <settings>
-<setting alwaysvectorfont="yes"/>
+<setting alwaysvectorfont="no"/>
 <setting verticaltext="up"/>
 </settings>
@@
 <layers>
 <layer number="1" name="Top" color="4" fill="1" visible="yes" active="yes"/>
-<layer number="2" name="Route2" color="1" fill="3" visible="no" active="yes"/>
+<layer number="2" name="Route2" color="1" fill="3" visible="yes" active="yes"/>
 <layer number="3" name="Route3" color="4" fill="3" visible="no" active="yes"/>
 <layer number="4" name="Route4" color="1" fill="4" visible="no" active="yes"/>
@@
 </element>
 <element name="D3" library="adafruit" library_urn="urn:adsk.eagle:library:420" package="SOD-123" package3d_urn="urn:adsk.eagle:package:6240753/1" value="" x="10.16" y="2.54" smashed="yes">
-<attribute name="NAME" x="9.06" y="3.54" size="0.4064" layer="25"/>
 <attribute name="VALUE" x="9.06" y="1.256" size="0.4064" layer="27"/>
 </element>
@@
 <attribute name="MF" value="Diodes Inc." x="21.59" y="2.54" size="1.778" layer="27" display="off"/>
 <attribute name="MP" value="BZT52C3V9-7-F" x="21.59" y="2.54" size="1.778" layer="27" display="off"/>
-<attribute name="NAME" x="19.39" y="3.84" size="0.8128" layer="25"/>
 <attribute name="PACKAGE" value="SOD-123 Fairchild Semiconductor" x="21.59" y="2.54" size="1.778" layer="27" display="off"/>
 <attribute name="PRICE" value="None" x="21.59" y="2.54" size="1.778" layer="27" display="off"/>
@@
 <attribute name="MF" value="Diodes Inc." x="17.145" y="15.24" size="1.778" layer="27" display="off"/>
 <attribute name="MP" value="BZT52C3V9-7-F" x="17.145" y="15.24" size="1.778" layer="27" display="off"/>
-<attribute name="NAME" x="14.945" y="16.54" size="0.8128" layer="25"/>
 <attribute name="PACKAGE" value="SOD-123 Fairchild Semiconductor" x="17.145" y="15.24" size="1.778" layer="27" display="off"/>
 <attribute name="PRICE" value="None" x="17.145" y="15.24" size="1.778" layer="27" display="off"/>
@@
 <contactref element="D5" pad="A"/>
 <contactref element="D4" pad="A"/>
-<wire x1="23.27" y1="2.54" x2="18.825" y2="15.24" width="0" layer="19" extent="1-1"/>
-<wire x1="6.41" y1="12.39" x2="23.27" y2="2.54" width="0" layer="19" extent="1-1"/>
 </signal>
 <signal name="+5V">
@@
 <contactref element="C2" pad="1"/>
 <contactref element="C1" pad="1"/>
-<wire x1="36.41" y1="15.24" x2="36.41" y2="12.7" width="0.254" layer="16"/>
-<wire x1="36.41" y1="12.7" x2="41.91" y2="12.7" width="0.254" layer="16"/>
 <wire x1="41.49" y1="15.24" x2="41.91" y2="14.82" width="0.254" layer="16"/>
 <wire x1="41.91" y1="14.82" x2="41.91" y2="12.7" width="0.254" layer="16"/>
@@
 <wire x1="49.53" y1="11.43" x2="48.26" y2="12.7" width="0.2032" layer="1"/>
 <wire x1="48.26" y1="12.7" x2="41.91" y2="12.7" width="0.2032" layer="1"/>
-<wire x1="35.56" y1="13.97" x2="38.1" y2="11.43" width="0.2032" layer="16"/>
-<wire x1="38.1" y1="11.43" x2="40.64" y2="11.43" width="0.2032" layer="16"/>
-<wire x1="40.64" y1="11.43" x2="41.91" y2="12.7" width="0.2032" layer="16"/>
 <wire x1="18.61" y1="5.955" x2="20.275" y2="7.62" width="0.2032" layer="1"/>
 <wire x1="20.275" y1="7.62" x2="20.32" y2="7.62" width="0.2032" layer="1"/>
@@
 <wire x1="38.8761125" y1="9.0311125" x2="41.91" y2="12.065" width="0.2032" layer="16"/>
 <wire x1="41.91" y1="12.065" x2="41.91" y2="12.7" width="0.2032" layer="16"/>
+<wire x1="36.41" y1="15.24" x2="38.95" y2="12.7" width="0.2032" layer="16"/>
+<wire x1="38.95" y1="12.7" x2="41.91" y2="12.7" width="0.2032" layer="16"/>
 <wire x1="19.05" y1="8.255" x2="20.32" y2="7.62" width="0" layer="19" extent="1-1"/>
 </signal>
@@
 <wire x1="9.89" y1="7.89" x2="10.16" y2="7.62" width="0.2032" layer="1"/>
 <wire x1="10.16" y1="7.62" x2="11.7" y2="7.62" width="0.2032" layer="1"/>
-<wire x1="11.7" y1="12.7" x2="10.16" y2="12.7" width="0.2032" layer="1"/>
-<wire x1="10.16" y1="12.7" x2="8.89" y2="11.43" width="0.2032" layer="1"/>
 <via x="8.89" y="11.43" extent="1-16" drill="0.35"/>
 <wire x1="8.89" y1="11.43" x2="8.89" y2="6.985" width="0.2032" layer="16"/>
@@
 <wire x1="7.315" y1="6.985" x2="6.41" y2="7.89" width="0.2032" layer="1"/>
 <contactref element="D5" pad="C"/>
-<wire x1="14.24" y1="15.24" x2="15.465" y2="15.24" width="0.2032" layer="1"/>
-<wire x1="11.7" y1="12.7" x2="14.24" y2="15.24" width="0.2032" layer="1"/>
+<wire x1="15.465" y1="15.24" x2="11.43" y2="15.24" width="0.2032" layer="1"/>
+<wire x1="11.43" y1="15.24" x2="8.89" y2="12.7" width="0.2032" layer="1"/>
+<wire x1="8.89" y1="12.7" x2="8.89" y2="11.43" width="0.2032" layer="1"/>
+<wire x1="11.7" y1="12.7" x2="10.43" y2="11.43" width="0.2032" layer="1"/>
+<wire x1="10.43" y1="11.43" x2="8.89" y2="11.43" width="0.2032" layer="1"/>
 </signal>
 <signal name="N$5">
@@
 <wire x1="18.415" y1="2.54" x2="16.51" y2="4.445" width="0.2032" layer="1"/>
 <wire x1="16.51" y1="7.62" x2="15.24" y2="8.89" width="0.2032" layer="1"/>
-<wire x1="15.24" y1="8.89" x2="12.7" y2="8.89" width="0.2032" layer="1"/>
-<wire x1="12.7" y1="8.89" x2="11.7" y2="9.89" width="0.2032" layer="1"/>
 <wire x1="11.7" y1="9.89" x2="11.7" y2="10.16" width="0.2032" layer="1"/>
 <wire x1="16.51" y1="4.445" x2="16.51" y2="7.62" width="0.2032" layer="1"/>
 <wire x1="6.68" y1="10.16" x2="6.41" y2="9.89" width="0.2032" layer="1"/>
-<wire x1="11.7" y1="10.16" x2="6.68" y2="10.16" width="0.2032" layer="1"/>
 <contactref element="D4" pad="C"/>
 <wire x1="19.91" y1="2.54" x2="18.415" y2="2.54" width="0.2032" layer="1"/>
+<wire x1="7.41" y1="8.89" x2="6.41" y2="9.89" width="0.2032" layer="1"/>
+<wire x1="15.24" y1="8.89" x2="9.525" y2="8.89" width="0.2032" layer="1"/>
+<wire x1="9.525" y1="8.89" x2="7.41" y2="8.89" width="0.2032" layer="1"/>
+<wire x1="11.7" y1="10.16" x2="10.795" y2="10.16" width="0.2032" layer="1"/>
+<wire x1="10.795" y1="10.16" x2="9.525" y2="8.89" width="0.2032" layer="1"/>
 </signal>
 <signal name="N$2">
@@
 <mfgpreviewcolor name="substratecolor" color="0xFF786E46"/>
 </mfgpreviewcolors>
+<errors>
+</errors>
 </board>
 </drawing>
